File: hardware/irl2fa.kicad_sch (KiCad schematic)
At the start: 51 parts, among them J1 FH34SRJ-24S, J3 TC2030-NL, Q1 AO3401A, Q2 AO3401A, Q3 Si1308EDL, Q4 AO3400A, Q5 VEMT2523SLX01, SW1 SKRHABE010, U1 STM32U083KCU6, U2 RV-3032-C7

Commit message: Make the fob smaller: 80.9 x 34.9 x 11.0 mm case, 77 x 31 x 0.8 mm board
The 7.5 mm BS-24-B4AA016 holder set the case thickness. Replace it with
the MYOUNG MY-2450-01 CR2450 clip (LCSC C964845, 5.70 mm, 5355 in stock,
$0.17): a sprung plate over the cell, with a bare 12 mm ENIG pad under
it as the negative contact. Same cell, so the battery-life budget is
unchanged.

- Board 80 x 34 x 1.0 -> 77 x 31 x 0.8 mm, corner radius 2.6, holes at
  the corner centres. Glass 0.9 mm from the long edges, 0.4 mm clear of
  the case's screw bosses; joystick 1.2 mm from the glass.
- Case 83.9 x 37.9 x 13.0 -> 80.9 x 34.9 x 11.0 mm (keep-out 7.6 -> 5.8).
- New footprint and model for the clip, drawn from drawing MY-CP-0106.
  The courtyard is the union of plate, cell and pads. The SKRH courtyard
  now follows body and pads instead of their bounding box.
- The cell slides in from the bottom edge. Rule area: no vias under the
  cell. J1 keeps its FPC insertion offset on the thinner board.
- Re-placed and re-routed (Freerouting 2.5): ERC/DRC 0 errors,
  0 unconnected. Fab outputs, case STL/3MF, renders and docs regenerated.
- Case tests take the skin samples above and below the window from
  board.yaml rather than fixed coordinates.

Co-Authored-By: Claude Opus 5.5 <noreply@anthropic.com>
Parts:
- BT1: footprint irl2fa:BatteryHolder_MYOUNG_BS-24-B4AA016_CR2450 -> irl2fa:BatteryHolder_MYOUNG_MY-2450-01_CR2450; LCSC C964809 -> C964845; MPN BS-24-B4AA016 -> MY-2450-01
Changed lines of the file:
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@@
 			)
 		)
-		(property "Footprint" "irl2fa:BatteryHolder_MYOUNG_BS-24-B4AA016_CR2450"
+		(property "Footprint" "irl2fa:BatteryHolder_MYOUNG_MY-2450-01_CR2450"
 			(at 205.74 45.72 0)
 			(effects
@@
 			)
 		)
-		(property "Datasheet" "https://www.lcsc.com/product-detail/C964809.html"
+		(property "Datasheet" "https://www.lcsc.com/product-detail/C964845.html"
 			(at 205.74 45.72 0)
 			(effects
@@
 			)
 		)
-		(property "Description" "CR2450 coin cell holder, SMT"
+		(property "Description" "CR2450 coin cell clip, SMT, 5.7 mm (the PCB pad is the - contact)"
 			(at 205.74 45.72 0)
 			(effects
@@
 			)
 		)
-		(property "LCSC" "C964809"
+		(property "LCSC" "C964845"
 			(at 205.74 45.72 0)
 			(effects
@@
 			)
 		)
-		(property "MPN" "BS-24-B4AA016"
+		(property "MPN" "MY-2450-01"
 			(at 205.74 45.72 0)
 			(effects

Commit message: WIP board fixes: parts, keep-outs, silkscreen, test pads, benches (board not yet routed)
Co-Authored-By: Claude Opus 5.5 <noreply@anthropic.com>
Parts:
- added TP3: SWDIO, TestPoint:TestPoint_Pad_D1.5mm, symbol Connector:TestPoint
- added TP4: SWCLK, TestPoint:TestPoint_Pad_D1.5mm, symbol Connector:TestPoint
- added TP5: NRST, TestPoint:TestPoint_Pad_D1.5mm, symbol Connector:TestPoint
- Q3: value Si1308EDL -> NX3008NBK; footprint Package_TO_SOT_SMD:SOT-323_SC-70 -> Package_TO_SOT_SMD:SOT-23; symbol Transistor_FET:Si1308EDL -> Transistor_FET:Q_NMOS_GSD; LCSC C469327 -> C179399; MPN Si1308EDL-T1-GE3 -> NX3008NBK,215; Manufacturer Vishay -> Nexperia
- Q5: value VEMT2523SLX01 -> VEMT2023SLX01; footprint irl2fa:PhotoTransistor_Vishay_VEMT2523SLX01_SideView -> irl2fa:PhotoTransistor_Vishay_VEMT2023SLX01_SideView; LCSC C511451 -> C2843576; MPN VEMT2523SLX01 -> VEMT2023SLX01
- R8: value 100 -> 68; LCSC C25076 -> C25131; MPN 0402WGF1000TCE -> 0402WGF680JTCE
- TP1, TP2: footprint TestPoint:TestPoint_Pad_D1.0mm -> TestPoint:TestPoint_Pad_D1.5mm
Connections:
- net GND: now also SW1.MP
- net NRST: now also TP5.1
- net SWCLK: now also TP4.1
- net SWDIO: now also TP3.1
- no-connect marks 13 -> 12
Other:
- moved on the sheet: Q5, R10, R9
